File: Sphale.kicad_sch (KiCad schematic)
At the start: 29 parts, among them J1 USB_C_Receptacle_USB2.0, J2 Conn_01x12, J3 Conn_01x12, J4 Conn_01x05, SW1 RESET, SW3 BOOT, U1 STM32F303CCTx, U2 RT9013-33GB, Y1 8MHz

Commit message: Update BOM and references
Parts:
- C1: renamed from C5; MFR. Part# (none) -> CL05A106MQ5NUNC
- C10: renamed from C7; MFR. Part# (none) -> 0402CG120J500NT
- C11, C12: MFR. Part# (none) -> CL05A105KA5NQNC
- C2: renamed from C4; LCSC C307331 -> C1525; MFR. Part# (none) -> CL05B104KO5NNNC
- C3: LCSC C307331 -> C1525; MFR. Part# (none) -> CL05B104KO5NNNC
- C4: renamed from C1; LCSC C307331 -> C1525; MFR. Part# (none) -> CL05B104KO5NNNC
- C5: renamed from C2; LCSC C307331 -> C1525; MFR. Part# (none) -> CL05B104KO5NNNC
- C6: renamed from C9; MFR. Part# (none) -> CL05B103KB5NNNC
- C7: renamed from C10; MFR. Part# (none) -> CL05A105KA5NQNC
- C8: renamed from C6; LCSC C307331 -> C1525; MFR. Part# (none) -> CL05B104KO5NNNC
- C9: renamed from C8; MFR. Part# (none) -> 0402CG120J500NT
- D1: MFR. Part# (none) -> B5817WS
- F1: MFR. Part# (none) -> SMD0805B050TF
- J4: renamed from J1; MFR. Part# (none) -> TYPE-C-31-M-12
- LD1: MFR. Part# (none) -> KT-0603R
- R1: renamed from R4; MFR. Part# (none) -> ARG02BTC1501
- R2: renamed from R1; MFR. Part# (none) -> 0402WGF1002TCE
- R3: renamed from R5; value 10k -> 5.1k; LCSC C25744 -> C25905; MFR. Part# (none) -> 0402WGF5101TCE
- R4: renamed from R2; MFR. Part# (none) -> 0402WGF5101TCE
- R5: renamed from R3; MFR. Part# (none) -> 0402WGF5101TCE
- SW1: LCSC C231329 -> C498294; MFR. Part# (none) -> TS-1064S-A1B2-D4
- SW2: renamed from SW3; LCSC C231329 -> C498294; MFR. Part# (none) -> TS-1064S-A1B2-D4
- U1: MFR. Part# (none) -> STM32F303CCT6
- U2: LCSC C47773 -> C587158; MFR. Part# (none) -> TPRT9013-33GB
- Y1: MFR. Part# (none) -> X32258MSB4SI
- renumbered J2 to J1, J3 to J2, J4 to J3
Other:
- company: The Pro Micro compatible STM32 board -> SideraKB
- moved on the sheet: LD1, R3
